File: moPsy_Rectifier/moPsy_Rectifier.kicad_pcb (KiCad board)
At the start: 2 copper layers, 41 parts, among them J1 Conn_01x01_Male, J10 Conn_01x01_Male, J11 Conn_01x01_Male, J12 Conn_01x03_Male, J13 Conn_01x08_Male, J14 Conn_01x01_Male, J15 Conn_01x01_Male, J16 Conn_01x01_Male, J17 Conn_01x01_Male, J2 Conn_01x01_Male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

Commit message: PCB Layout
Parts:
- added REF**: MountingHole_3.2mm_M3, MountingHole:MountingHole_3.2mm_M3, F.Cu at (39.4, 27.9)
- added REF**: MountingHole_3.2mm_M3, MountingHole:MountingHole_3.2mm_M3, F.Cu at (162.6, 90.2)
- added REF**: MountingHole_3.2mm_M3, MountingHole:MountingHole_3.2mm_M3, F.Cu at (163.8, 27.9)
- added REF**: MountingHole_3.2mm_M3, MountingHole:MountingHole_3.2mm_M3, F.Cu at (39.4, 90.2)
- added Ref**: Val**, moPsy_KiCad:moPsy_logo_kicad_20x09_FSilk, F.Cu at (114.3, 34.9)
- moved D2 162.0 mm to (48.3, 54.6)
- moved D1 154.3 mm to (48.3, 62.2)
- moved R2 149.6 mm to (44.5, 54.6), turned to 90 degrees
- moved R1 141.5 mm to (44.5, 62.2), turned to -90 degrees
- moved R4 124.4 mm to (141.0, 34.3), turned to 180 degrees
- moved D6 123.3 mm to (154.9, 36.8), turned to 90 degrees
- moved D5 116.3 mm to (147.3, 36.8), turned to 90 degrees
- moved R3 110.9 mm to (141.0, 38.1), turned to 180 degrees
- moved J3 110.2 mm to (39.3, 49.5), turned to 90 degrees
- moved R5 107.0 mm to (85.1, 49.0), turned to -90 degrees
- moved J5 102.2 mm to (55.9, 56.5)
- moved J8 95.8 mm to (76.2, 29.5), turned to 90 degrees
- moved J14 94.8 mm to (165.1, 40.7), turned to 90 degrees
- moved C1 94.7 mm to (143.5, 57.1), turned to 90 degrees
- moved C3 94.7 mm to (118.1, 57.1), turned to 90 degrees
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Routing:
- net -15V_PWR: track 0.00 -> 174.8 mm
- net -15V: track 0.00 -> 157.6 mm
- net +15V: track 0.00 -> 144.7 mm
- net -15V_SW: track 0.00 -> 114.7 mm
- net LED_CHARGING: track 0.00 -> 97.8 mm
- net +15V_SW: track 0.00 -> 92.8 mm
- net +15V_PWR: track 0.00 -> 71.6 mm
- net REL_RETURN: track 0.00 -> 60.4 mm
- net REL_Charge: track 0.00 -> 58.4 mm
- net REL_PwrGood: track 0.00 -> 47.8 mm
- net Net-(D3-Pad3): track 0.00 -> 32.9 mm
- net Net-(D4-Pad3): track 0.00 -> 30.2 mm
- net Net-(F1-Pad2): track 0.00 -> 21.9 mm
- net Net-(F2-Pad2): track 0.00 -> 18.6 mm
- net Net-(D4-Pad4): track 0.00 -> 18.2 mm
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- added copper zone on B.Cu, net GND
- added copper zone on F.Cu, net GND
Other:
- board outline added: 134.6 x 72.4 mm
- board text added: "+15V"
- board text added: "+15V Amp"
- board text added: "-15V"
- board text added: "-15V Amp"
- board text added: "-CHRG"
- board text added: "-GOOD"
- board text added: "1"
- board text added: "CHRG"
- board text added: "GND"
- board text added: "GOOD"
- board text added: "RET"
- board text added: "Vin 1"
- board text added: "Vin 2"

Commit message: Finishing and Roundes Corners
Parts:
- moved REF** 1.27 mm to (163.8, 90.2)
Routing:
- net -15V_PWR: track 174.8 -> 175.9 mm
Other:
- outline, holes or cut-outs redrawn
- board text added: "IN"
- board text added: "OUT"
Changed lines of the file:
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@@
   )
   (footprint "MountingHole:MountingHole_3.2mm_M3" (layer "F.Cu")
-    (at 162.56 90.17)
+    (at 163.83 90.17)
     (descr "Mounting Hole 3.2mm, no annular, M3")
     (tags "mounting hole 3.2mm no annular m3")
@@
       (net 2 "GND") (pinfunction "Pin_1") (pintype "passive"))
   )
-  (gr_rect (start 34.29 22.86) (end 168.91 95.25) (layer "Edge.Cuts") (width 0.1) (fill none))
+  (gr_arc (start 168.91 92.71) (mid 168.166051 94.506051) (end 166.37 95.25) (layer "Edge.Cuts") (width 0.1))
+  (gr_arc (start 166.37 22.86) (mid 168.166051 23.603949) (end 168.91 25.4) (layer "Edge.Cuts") (width 0.1))
+  (gr_line (start 34.29 92.71) (end 34.29 25.4) (layer "Edge.Cuts") (width 0.1))
+  (gr_arc (start 34.29 25.4) (mid 35.033949 23.603949) (end 36.83 22.86) (layer "Edge.Cuts") (width 0.1))
+  (gr_arc (start 36.83 95.25) (mid 35.033949 94.506051) (end 34.29 92.71) (layer "Edge.Cuts") (width 0.1))
+  (gr_line (start 36.83 22.86) (end 166.37 22.86) (layer "Edge.Cuts") (width 0.1))
+  (gr_line (start 168.91 25.4) (end 168.91 92.71) (layer "Edge.Cuts") (width 0.1))
+  (gr_line (start 166.37 95.25) (end 36.83 95.25) (layer "Edge.Cuts") (width 0.1))
   (gr_text "+15V Amp" (at 73.025 46.355 90) (layer "F.SilkS")
     (effects (font (size 1 1) (thickness 0.15)))
@@
     (effects (font (size 1 1) (thickness 0.15)))
   )
+  (gr_text "IN" (at 78.74 66.04 90) (layer "F.SilkS")
+    (effects (font (size 1 1) (thickness 0.15)))
+  )
   (gr_text "GND" (at 167.64 53.34 90) (layer "F.SilkS")
     (effects (font (size 1 1) (thickness 0.15)))
@@
     (effects (font (size 1 1) (thickness 0.15)))
   )
+  (gr_text "OUT" (at 78.74 77.47 90) (layer "F.SilkS")
+    (effects (font (size 1 1) (thickness 0.15)))
+  )
   (gr_text "-15V" (at 55.88 65.405 90) (layer "F.SilkS")
     (effects (font (size 1 1) (thickness 0.15)))
@@
     (effects (font (size 1 1) (thickness 0.15)))
   )
+  (gr_text "OUT" (at 78.74 40.64 90) (layer "F.SilkS")
+    (effects (font (size 1 1) (thickness 0.15)))
+  )
   (gr_text "+15V" (at 44.45 57.15) (layer "F.SilkS")
     (effects (font (size 1 1) (thickness 0.15)))
@@
   )
   (gr_text "GND" (at 167.64 66.08 90) (layer "F.SilkS")
+    (effects (font (size 1 1) (thickness 0.15)))
+  )
+  (gr_text "IN" (at 78.74 52.07 90) (layer "F.SilkS")
     (effects (font (size 1 1) (thickness 0.15)))
   )
@@
   (segment (start 76.2 74.97) (end 82.55 68.62) (width 0.6096) (layer "B.Cu") (net 17))
   (segment (start 82.55 68.62) (end 82.55 37.514003) (width 0.6096) (layer "B.Cu") (net 17))
+  (segment (start 100.86 83.26) (end 114.27 69.85) (width 1.524) (layer "F.Cu") (net 18))
   (segment (start 135.794511 26.765489) (end 155.035489 26.765489) (width 0.25) (layer "F.Cu") (net 18))
-  (segment (start 159.98 71.12) (end 165.1 76.24) (width 1.524) (layer "F.Cu") (net 18))
   (segment (start 165.1 76.24) (end 165.1 81.24) (width 1.524) (layer "F.Cu") (net 18))
-  (segment (start 100.86 83.26) (end 113 71.12) (width 1.524) (layer "F.Cu") (net 18))
   (segment (start 128.27 34.29) (end 135.794511 26.765489) (width 0.25) (layer "F.Cu") (net 18))
-  (segment (start 113 71.12) (end 159.98 71.12) (width 1.524) (layer "F.Cu") (net 18))
+  (segment (start 114.27 69.85) (end 158.71 69.85) (width 1.524) (layer "F.Cu") (net 18))
+  (segment (start 158.71 69.85) (end 165.1 76.24) (width 1.524) (layer "F.Cu") (net 18))
   (segment (start 155.035489 26.765489) (end 156.21 27.94) (width 0.25) (layer "F.Cu") (net 18))
   (segment (start 160.02 71.16) (end 165.1 76.24) (width 0.25) (layer "B.Cu") (net 18))
