File: moPsy_Rectifier/moPsy_Rectifier.kicad_pcb (KiCad board)
At the start: 2 copper layers, 134.6 x 72.4 mm, 46 parts, among them J1 Conn_01x01_Male, J10 Conn_01x01_Male, J11 Conn_01x01_Male, J12 Conn_01x03_Male, J13 Conn_01x08_Male, J14 Conn_01x01_Male, J15 Conn_01x01_Male, J16 Conn_01x01_Male, J17 Conn_01x01_Male, J2 Conn_01x01_Male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

Commit message: Add OSHW logo to Rectifier PCB
Parts:
- added REF**: OSHW-Logo2_7.3x6mm_SilkScreen, Symbol:OSHW-Logo2_7.3x6mm_SilkScreen, F.Cu at (135.3, 27.9)

Commit message: Fix direction of V+ Pwr indicator LED
Parts:
- moved D2 2.54 mm to (50.8, 54.6), turned to 180 degrees
Connections:
- D2 pad 1: Net-(D2-Pad1) -> GND
- D2 pad 2: GND -> Net-(D2-Pad2)
- R2 pad 1: Net-(D2-Pad1) -> Net-(D2-Pad2)
Routing:
- net Net-(D2-Pad2): track 0.00 -> 3.81 mm
- net Net-(D2-Pad1): track 3.81 -> 0.00 mm
Changed lines of the file:
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@@
   (net 3 "-15V_SW")
   (net 4 "Net-(D1-Pad1)")
-  (net 5 "Net-(D2-Pad1)")
+  (net 5 "Net-(D2-Pad2)")
   (net 6 "Net-(D3-Pad3)")
   (net 7 "Net-(D3-Pad2)")
@@
   )
   (footprint "LED_THT:LED_D5.0mm" (layer "F.Cu")
-    (at 48.26 54.61)
+    (at 50.8 54.61 180)
     (descr "LED, diameter 5.0mm, 2 pins, http://cdn-reichelt.de/documents/datenblatt/A500/LL-504BC2E-009.pdf")
     (tags "LED diameter 5.0mm 2 pins")
@@
     (property "Sheetname" "")
     (attr through_hole)
-    (fp_text reference "D2" (at 5.08 -2.54) (layer "F.SilkS")
+    (fp_text reference "D2" (at -2.54 -2.5) (layer "F.SilkS")
       (effects (font (size 1 1) (thickness 0.15)))
     )
@@
     (fp_arc (start -1.23 -1.469694) (mid 4.17 0.000016) (end -1.230016 1.469666) (layer "F.Fab") (width 0.1))
     (fp_circle (center 1.27 0) (end 3.77 0) (layer "F.Fab") (width 0.1) (fill none))
-    (pad "1" thru_hole rect locked (at 0 0) (size 1.8 1.8) (drill 0.9) (layers *.Cu *.Mask)
-      (net 5 "Net-(D2-Pad1)") (pinfunction "K") (pintype "passive"))
-    (pad "2" thru_hole circle locked (at 2.54 0) (size 1.8 1.8) (drill 0.9) (layers *.Cu *.Mask)
-      (net 2 "GND") (pinfunction "A") (pintype "passive"))
+    (pad "1" thru_hole rect locked (at 0 0 180) (size 1.8 1.8) (drill 0.9) (layers *.Cu *.Mask)
+      (net 2 "GND") (pinfunction "K") (pintype "passive"))
+    (pad "2" thru_hole circle locked (at 2.54 0 180) (size 1.8 1.8) (drill 0.9) (layers *.Cu *.Mask)
+      (net 5 "Net-(D2-Pad2)") (pinfunction "A") (pintype "passive"))
     (model "${KICAD6_3DMODEL_DIR}/LED_THT.3dshapes/LED_D5.0mm.wrl"
       (offset (xyz 0 0 0))
@@
     (fp_line (start 1.85 -1.6) (end 1.85 1.6) (layer "F.Fab") (width 0.1))
     (pad "1" thru_hole circle locked (at 0 0 90) (size 1.6 1.6) (drill 0.8) (layers *.Cu *.Mask)
-      (net 5 "Net-(D2-Pad1)") (pintype "passive"))
+      (net 5 "Net-(D2-Pad2)") (pintype "passive"))
     (pad "2" thru_hole oval locked (at 12.7 0 90) (size 1.6 1.6) (drill 0.8) (layers *.Cu *.Mask)
       (net 16 "+15V") (pintype "passive"))
