File: moPsy_CapCharger_I/moPsy_CapCharger_I.kicad_pcb (KiCad board)
At the start: 2 copper layers, 30 x 31 mm, 12 parts, among them J1 Conn_01x08_Male, U1 LM79L12_TO92, U2 LM555xN

Commit message: Convert to KiCAD 6
Other:
- net class Default removed
