File: moPsy_Regulator_12Vpos/moPsy_Regulator_12Vpos.kicad_pcb (KiCad board)
At the start: 2 copper layers, 41 x 40 mm, 19 parts, among them J1 Conn_01x01_Male, J2 Conn_01x01_Male, J3 Conn_01x01_Male, J4 Conn_01x01_Male, U1 LT1084-ADJ

Commit message: Add OSHW logo to Regulator 12V pos PCB
Parts:
- added REF**: OSHW-Logo2_7.3x6mm_SilkScreen, Symbol:OSHW-Logo2_7.3x6mm_SilkScreen, B.Cu at (117.5, 63.5)
