File: moPsy_BusBoard_2/mopsy_BusBoard_2.kicad_pcb (KiCad board)
At the start: 2 copper layers, 238 x 24 mm, 29 parts, among them J1 Conn_02x08_Odd_Even, J101 Conn_01x01_Male, J102 Conn_01x01_Male, J103 Conn_01x01_Male, J104 Conn_01x01_Male, J105 Conn_01x01_Male, J106 Conn_01x01_Male, J107 Conn_01x01_Male, J108 Conn_01x01_Male, J109 Conn_01x01_Male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

Commit message: Add OSHW logo to BusBoard 2 PCB
Parts:
- added REF**: OSHW-Logo2_7.3x6mm_SilkScreen, Symbol:OSHW-Logo2_7.3x6mm_SilkScreen, F.Cu at (67.9, 81.9)
Other:
- net class Default removed
- net class PWR removed
- net class SIG removed
